File: KiCad/fightstick_pcb/fightstick_pcb.kicad_sch (KiCad schematic)
At the start: 93 parts, among them J1 USB_B_Micro, J2 Conn_01x02, J3 Conn_01x02, J4 Screw_Terminal_01x12, J5 Screw_Terminal_01x12, J6 Screw_Terminal_01x12, SW1 SW_Push, U1 SN74LVC1G14DBV, U10 SN74LVC1G14DBV, U11 SN74LVC1G14DBV, U12 SN74LVC1G14DBV, U13 SN74LVC1G14DBV, U14 SN74LVC1G14DBV, U15 SN74LVC1G14DBV, U2 SN74LVC1G14DBV, U3 NCP1117-3.3_SOT223, U4 W25Q128JVS, U5 SN74LVC1G14DBV, U6 SN74LVC1G14DBV, U7 SN74LVC1G14DBV, U8 SN74LVC1G14DBV, U9 RP2040, Y1 ABM8-272-T3

Commit message: PCB V1.2
Il n'y a plus de condensateurs polarisés
Parts:
- removed C18: 1u, Capacitor_SMD:CP_Elec_4x3, symbol Device:C_Polarized_US
- added C14, C15, C23, C24, C34, C35, C43, C44, C51, C52, C6, C7: 0.1u, Capacitor_SMD:C_0805_2012Metric, symbol Device:C
- added C16, C17, C25, C26, C30, C37, C38, C46, C47, C53, C54, C8, C9: 1u, Capacitor_SMD:C_0805_2012Metric, symbol Device:C
- renumbered C6 to C10, C7 to C11, C8 to C12, C9 to C13, C10 to C18, C11 to C19, C12 to C20, C13 to C21, C14 to C22, C15 to C27, C16 to C28, C17 to C29, C19 to C31, C20 to C32, C21 to C33, C22 to C36, C23 to C39, C24 to C40, C25 to C41, C26 to C42, C27 to C45, C28 to C48, C29 to C49, C30 to C50
Connections:
- net +3V3: now also C14.1, C15.1, C16.1, C17.1, C23.1, C24.1, C25.1, C26.1, C34.1, C35.1, C37.1, C38.1, C43.1, C44.1, C46.1, C47.1, C51.1, C52.1, C53.1, C54.1, C6.1, C7.1, C8.1, C9.1
- net GND: now also C14.2, C15.2, C16.2, C17.2, C23.2, C24.2, C25.2, C26.2, C30.2, C34.2, C35.2, C37.2, C38.2, C43.2, C44.2, C46.2, C47.2, C51.2, C52.2, C53.2, C54.2, C6.2, C7.2, C8.2, C9.2
- net LED_P2+: now also J6.5 (Pin_5); no longer J6.6 (Pin_6)
- net LED_P3+: now also J6.9 (Pin_9); no longer J6.10 (Pin_10)
- net LED_P3-: now also J6.8 (Pin_8); no longer J6.9 (Pin_9)
- net SW_1: now also J6.10 (Pin_10); no longer J6.8 (Pin_8)
- net SW_SELECT: now also J6.6 (Pin_6); no longer J6.5 (Pin_5)
- net at R19.2, U10.2: now also C30.1
Other:
- moved on the sheet: C12, C22, C31, C4, C42, C49, R11, R14, R16, R18, R2, R20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

Commit message: PCB V1.2.1
Tous les condensateurs et résistances sont maintenant plus gros
Parts:
- C1, C13, C18, C19, C2, C20, C27, C28, C29, C32, C33, C36, C39, C40: footprint Capacitor_SMD:C_0402_1005Metric -> Capacitor_SMD:C_0805_2012Metric
- R21, R22, R5, R6, R7: footprint Resistor_SMD:R_0402_1005Metric -> Resistor_SMD:R_0805_2012Metric
Other:
- note added: "Make sure C20 is close to pin 45 of RP2040"
- note added: "Make sure C28 is close to pin 44 of RP2040"
- note removed: "Make sure C12 is close to pin 45 of RP2040"
- note removed: "Make sure C16 is close to pin 44 of RP2040"
Changed lines of the file:
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@@
 		)
 	)
-	(text "Make sure C12 is close to pin 45 of RP2040"
+	(text "Make sure C20 is close to pin 45 of RP2040"
 		(exclude_from_sim no)
 		(at 107.442 155.448 0)
@@
 		)
 	)
-	(text "Make sure C16 is close to pin 44 of RP2040"
+	(text "Make sure C28 is close to pin 44 of RP2040"
 		(exclude_from_sim no)
 		(at 218.44 156.21 0)
@@
 			)
 		)
-		(property "Footprint" "Resistor_SMD:R_0402_1005Metric"
+		(property "Footprint" "Resistor_SMD:R_0805_2012Metric"
 			(at 61.722 196.85 90)
 			(effects
@@
 			)
 		)
-		(property "Footprint" "Resistor_SMD:R_0402_1005Metric"
+		(property "Footprint" "Resistor_SMD:R_0805_2012Metric"
 			(at 48.26 210.312 90)
 			(effects
@@
 			)
 		)
-		(property "Footprint" "Capacitor_SMD:C_0402_1005Metric"
+		(property "Footprint" "Capacitor_SMD:C_0805_2012Metric"
 			(at 105.1052 196.85 0)
 			(effects
@@
 			)
 		)
-		(property "Footprint" "Resistor_SMD:R_0402_1005Metric"
+		(property "Footprint" "Resistor_SMD:R_0805_2012Metric"
 			(at 232.41 167.132 90)
 			(effects
@@
 			)
 		)
-		(property "Footprint" "Resistor_SMD:R_0402_1005Metric"
+		(property "Footprint" "Resistor_SMD:R_0805_2012Metric"
 			(at 232.41 174.752 90)
 			(effects
@@
 			)
 		)
-		(property "Footprint" "Capacitor_SMD:C_0402_1005Metric"
+		(property "Footprint" "Capacitor_SMD:C_0805_2012Metric"
 			(at 211.7852 142.24 0)
 			(effects
@@
 			)
 		)
-		(property "Footprint" "Capacitor_SMD:C_0402_1005Metric"
+		(property "Footprint" "Capacitor_SMD:C_0805_2012Metric"
 			(at 223.2152 142.24 0)
 			(effects
@@
 			)
 		)
-		(property "Footprint" "Capacitor_SMD:C_0402_1005Metric"
+		(property "Footprint" "Capacitor_SMD:C_0805_2012Metric"
 			(at 234.6452 142.24 0)
 			(effects
@@
 			)
 		)
-		(property "Footprint" "Capacitor_SMD:C_0402_1005Metric"
+		(property "Footprint" "Capacitor_SMD:C_0805_2012Metric"
 			(at 246.0752 142.24 0)
 			(effects
@@
 			)
 		)
-		(property "Footprint" "Capacitor_SMD:C_0402_1005Metric"
+		(property "Footprint" "Capacitor_SMD:C_0805_2012Metric"
 			(at 257.5052 142.24 0)
 			(effects
@@
 			)
 		)
-		(property "Footprint" "Capacitor_SMD:C_0402_1005Metric"
+		(property "Footprint" "Capacitor_SMD:C_0805_2012Metric"
 			(at 268.9352 142.24 0)
 			(effects
@@
 			)
 		)
-		(property "Footprint" "Capacitor_SMD:C_0402_1005Metric"
+		(property "Footprint" "Capacitor_SMD:C_0805_2012Metric"
 			(at 280.3652 142.24 0)
 			(effects
@@
 			)
 		)
-		(property "Footprint" "Capacitor_SMD:C_0402_1005Metric"
+		(property "Footprint" "Capacitor_SMD:C_0805_2012Metric"
 			(at 145.7452 142.24 0)
 			(effects
@@
 			)
 		)
-		(property "Footprint" "Capacitor_SMD:C_0402_1005Metric"
+		(property "Footprint" "Capacitor_SMD:C_0805_2012Metric"
 			(at 157.1752 142.24 0)
 			(effects
@@
 			)
 		)
-		(property "Footprint" "Capacitor_SMD:C_0402_1005Metric"
+		(property "Footprint" "Capacitor_SMD:C_0805_2012Metric"
 			(at 157.1752 157.48 0)
 			(effects
@@
 			)
 		)
-		(property "Footprint" "Capacitor_SMD:C_0402_1005Metric"
+		(property "Footprint" "Capacitor_SMD:C_0805_2012Metric"
 			(at 211.7852 157.48 0)
 			(effects
@@
 			)
 		)
-		(property "Footprint" "Capacitor_SMD:C_0402_1005Metric"
+		(property "Footprint" "Capacitor_SMD:C_0805_2012Metric"
 			(at 31.75 257.5052 0)
 			(effects
@@
 			)
 		)
-		(property "Footprint" "Resistor_SMD:R_0402_1005Metric"
+		(property "Footprint" "Resistor_SMD:R_0805_2012Metric"
 			(at 68.58 264.922 90)
 			(effects
@@
 			)
 		)
-		(property "Footprint" "Capacitor_SMD:C_0402_1005Metric"
+		(property "Footprint" "Capacitor_SMD:C_0805_2012Metric"
 			(at 31.75 267.6652 0)
 			(effects
